File: HCCentral/Board/HCCentral.kicad_pcb (KiCad board)
At the start: 2 copper layers, 100.1 x 99.8 mm, 68 parts, among them CON1 BARREL_JACK, CON2 SD_Card, IC1 ENC28J60-I/SO, IC2 ATMEGA1284P-A, J1 RJ45-TRJ0011BANL, P2 ANT_433, P3 ANT_866, P4 ISP, P6 SPI, P7 UART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

Commit message: Deleted Gerbers, Updated V1.5
Parts:
- C11: value 10nF -> 100nF
- R10: value R -> 15k
- R13, R14: value 180R -> 1kR
- R7: value 2k -> 2k32
Connections:
- IC2 pad 32: (no net) -> /Controller_USB_SD/IRQ_LAN
- IC2 pad 44: /Controller_USB_SD/IRQ_LAN -> (no net)
Routing:
- net /Controller_USB_SD/IRQ_LAN: track 74.6 -> 91.3 mm, vias 2 -> 6
- net +3V3: track 376.2 -> 366.7 mm
- net GND: track 502.6 -> 498.8 mm
- net Net-(IC1-Pad27): track 47.7 -> 46.1 mm
Other:
- board text added: "v1.5 D. Walter"
- board text removed: "v1.0 D. Walter"
